Commit message: Modify the specifications of the range sensor

File: model/mobile_robot_sensors.urdf (robot description, URDF)
Before this commit: robot MobileRobot, 7 links, 6 joints
Links:
- removed link VLP_16
- added link LiDAR; visual cylinder length=0.03 radius=0.05
- link RealSense: geometry visual box size=0.064 0.022 0.024; visual cylinder length=0.024 radius=0.011
Joints:
- removed joint VLP_16FixedJoint
- added joint LiDARFixedJoint: type fixed, parent TiltLink, child LiDAR, origin xyz=0 0 0.025
